Commit message: Update URDF for camera integration & setting bridge configuration

File: aruco_visual_servoing/urdf/aruco_bot_diff.gazebo.xacro (robot description, xacro)
@@ -30,4 +30,7 @@
         <odom_publish_frequency>30</odom_publish_frequency>
     </plugin>
+    <plugin filename="gz-sim-sensors-system" name="gz::sim::systems::Sensors">
+        <render_engine>ogre2</render_engine>
+    </plugin>
     <plugin filename="gz-sim-joint-state-publisher-system"
             name="gz::sim::systems::JointStatePublisher">
@@ -35,5 +38,5 @@
     </plugin>
   </gazebo>
-<gazebo reference="left_wheel">
+  <gazebo reference="left_wheel">
     <mu1>1.0</mu1>
     <mu2>1.0</mu2>
@@ -59,3 +62,33 @@
     <kd>1.0</kd>
   </gazebo>
+  <gazebo reference="camera_link">
+    <sensor name="camera" type="camera">
+      <camera>
+        <horizontal_fov>1.3962634</horizontal_fov>
+        <image>
+          <width>640</width>
+          <height>480</height>
+          <format>R8G8B8</format>
+        </image>
+        <clip>
+          <near>0.1</near>
+          <far>15</far>
+        </clip>
+        <noise>
+          <type>gaussian</type>
+          <!-- Noise is sampled independently per pixel on each frame.
+               That pixel's noise value is added to each of its color
+               channels, which at that point lie in the range [0,1]. -->
+          <mean>0.0</mean>
+          <stddev>0.007</stddev>
+        </noise>
+        <optical_frame_id>camera_link_optical</optical_frame_id>
+        <camera_info_topic>camera/camera_info</camera_info_topic>
+      </camera>
+      <always_on>1</always_on>
+      <update_rate>20</update_rate>
+      <visualize>true</visualize>
+      <topic>camera/image</topic>
+    </sensor>
+  </gazebo>
 </robot>

File: aruco_visual_servoing/urdf/aruco_bot_diff.xacro (robot description, xacro)
@@ -122,4 +122,23 @@
     </inertial>
   </link>
+  <!-- Camera -->
+  <link name="camera_link">
+    <visual>
+      <geometry>
+        <box size="0.2 0.2 0.2"/>
+      </geometry>
+      <material name="blue"/>
+    </visual>
+    <collision>
+      <geometry>
+        <box size="0.2 0.2 0.2"/>
+      </geometry>
+    </collision>
+    <inertial>
+      <mass value="0.1"/>
+      <inertia ixx="0.001" ixy="0" ixz="0" iyy="0.001" iyz="0" izz="0.001"/>
+    </inertial>
+  </link>
+  <link name="camera_link_optical"/>
   <!-- Joints -->
   <joint name="left_wheel_joint" type="continuous">
@@ -142,3 +161,13 @@
     <origin xyz="0.8 0 -0.2" rpy="0 0 0"/>
   </joint>
+  <joint name="camera_joint" type="fixed">
+    <parent link="base_link"/>
+    <child link="camera_link"/>
+    <origin xyz="0.9 0 0.36" rpy="0 0 0"/>
+  </joint>
+  <joint type="fixed" name="camera_optical_joint">
+    <origin xyz="0 0 0" rpy="-${PI/2} 0 -${PI/2}"/>
+    <child link="camera_link_optical"/>
+    <parent link="camera_link"/>
+  </joint>
 </robot>
