Commit message: Add materials.xacro for standardized Gazebo-compatible materials

File: aruco_visual_servoing/urdf/aruco_bot_diff.xacro (robot description, xacro)
@@ -1,53 +1,52 @@
 <?xml version="1.0"?>
+<!--
+  ArUco Visual Servoing - Differential Drive Robot URDF
+  This file defines the complete kinematic and dynamic structure of a differential drive
+  mobile robot equipped with an onboard camera for ArUco marker-based visual servoing.
+  The model includes a base chassis, two independently actuated wheels, a caster wheel for
+  stability, and a mounted camera with proper optical frame alignment.
+  Robot Features:
+  - Differential drive locomotion with independent left/right wheel control
+  - Camera system with optical frame transformation
+  - Caster wheel for stability on uneven surfaces
+  - Complete inertial properties for physics simulation
+  Author: Mohamed Eyad
+  Date: December 13, 2025
+  License: See package.xml for license information
+-->
 <robot name="aruco_bot" xmlns:xacro="http://www.ros.org/wiki/xacro">
+  <!-- ========================================= -->
+  <!-- External File Includes                    -->
+  <!-- ========================================= -->
   <xacro:include filename="$(find aruco_visual_servoing)/urdf/aruco_bot_diff.gazebo.xacro"/>
-  <!-- Basic params -->
-  <xacro:property name="WHEEL_RADIUS" value="0.4"/> <!-- meters -->
-  <xacro:property name="WHEEL_WIDTH" value="0.2"/>
-  <xacro:property name="CASTER_RADIUS" value="0.2"/>
-  <xacro:property name="BASE_LENGTH" value="2.0"/>
-  <xacro:property name="BASE_WIDTH" value="1.0"/>
-  <xacro:property name="BASE_HEIGHT" value="0.5"/>
+  <xacro:include filename="$(find aruco_visual_servoing)/urdf/materials.xacro"/>
+  <!-- ========================================= -->
+  <!-- Robot Geometry Parameters                 -->
+  <!-- ========================================= -->
+  <xacro:property name="WHEEL_RADIUS" value="0.4"/>        <!-- meters -->
+  <xacro:property name="WHEEL_WIDTH" value="0.2"/>         <!-- meters -->
+  <xacro:property name="CASTER_RADIUS" value="0.2"/>       <!-- meters -->
+  <xacro:property name="BASE_LENGTH" value="2.0"/>         <!-- meters -->
+  <xacro:property name="BASE_WIDTH" value="1.0"/>          <!-- meters -->
+  <xacro:property name="BASE_HEIGHT" value="0.5"/>         <!-- meters -->
   <xacro:property name="WHEEL_SEPARATION" value="${BASE_WIDTH + WHEEL_WIDTH}"/>
-  <!-- Mass / inertia approximations -->
-  <xacro:property name="BASE_MASS" value="5.0"/>
-  <xacro:property name="WHEEL_MASS" value="2.0"/>
-  <xacro:property name="CASTER_MASS" value="1.0"/>
-  <!-- Mathematical constant -->
+  <!-- ========================================= -->
+  <!-- Robot Mass Properties                     -->
+  <!-- ========================================= -->
+  <xacro:property name="BASE_MASS" value="5.0"/>           <!-- kilograms -->
+  <xacro:property name="WHEEL_MASS" value="2.0"/>          <!-- kilograms -->
+  <xacro:property name="CASTER_MASS" value="1.0"/>         <!-- kilograms -->
+  <!-- ========================================= -->
+  <!-- Mathematical Constants                    -->
+  <!-- ========================================= -->
   <xacro:property name="PI" value="3.14159265359"/>
-  <!-- Material colors -->
-  <material name="black">
-    <color rgba="0.0 0.0 0.0 1.0"/>
-  </material>
-  <material name="white">
-    <color rgba="1.0 1.0 1.0 1.0"/>
-  </material>
-  <material name="red">
-    <color rgba="0.8 0.0 0.0 1.0"/>
-  </material>
-  <material name="blue">
-    <color rgba="0.0 0.0 0.8 1.0"/>
-  </material>
-  <material name="green">
-    <color rgba="0.0 0.8 0.0 1.0"/>
-  </material>
-  <material name="grey">
-    <color rgba="0.5 0.5 0.5 1.0"/>
-  </material>
-  <material name="silver">
-    <color rgba="0.75 0.75 0.75 1.0"/>
-  </material>
-  <material name="orange">
-    <color rgba="${255/255} ${108/255} ${10/255} 1.0"/>
-  </material>
-  <material name="brown">
-    <color rgba="${222/255} ${207/255} ${195/255} 1.0"/>
-  </material>
-  <!-- Chassis -->
+  <!-- ========================================= -->
+  <!-- Base Footprint and Chassis                -->
+  <!-- ========================================= -->
   <link name="base_footprint"/>
   <joint name="base_joint" type="fixed">
     <parent link="base_footprint"/>
     <child link="base_link"/>
-    <origin xyz="0.0 0 0" rpy="0 0 0.0" />
+    <origin xyz="0.0 0 0" rpy="0 0 0.0"/>
   </joint>
   <link name="base_link">
@@ -65,7 +64,10 @@
     <inertial>
       <mass value="${BASE_MASS}"/>
-        <inertia ixx="0.83333" ixy="0" ixz="0" iyy="1.66667" iyz="0" izz="1.66667"/>
+      <inertia ixx="0.83333" ixy="0" ixz="0" iyy="1.66667" iyz="0" izz="1.66667"/>
     </inertial>
   </link>
+  <!-- ========================================= -->
+  <!-- Wheel Links                               -->
+  <!-- ========================================= -->
   <!-- Left Wheel -->
   <link name="left_wheel">
@@ -104,5 +106,7 @@
     </inertial>
   </link>
-  <!-- Caster Wheel -->
+  <!-- ========================================= -->
+  <!-- Caster Wheel Link                         -->
+  <!-- ========================================= -->
   <link name="caster">
     <visual>
@@ -114,5 +118,5 @@
     <collision>
       <geometry>
-        <sphere radius="0.2"/>
+        <sphere radius="${CASTER_RADIUS}"/>
       </geometry>
     </collision>
@@ -122,5 +126,8 @@
     </inertial>
   </link>
-  <!-- Camera -->
+  <!-- ========================================= -->
+  <!-- Camera Links                              -->
+  <!-- ========================================= -->
+  <!-- Camera Physical Link -->
   <link name="camera_link">
     <visual>
@@ -140,6 +147,10 @@
     </inertial>
   </link>
+  <!-- Camera Optical Frame (aligned with camera sensor coordinate system) -->
   <link name="camera_link_optical"/>
-  <!-- Joints -->
+  <!-- ========================================= -->
+  <!-- Robot Joints                              -->
+  <!-- ========================================= -->
+  <!-- Left Wheel Joint (continuous rotation for locomotion) -->
   <joint name="left_wheel_joint" type="continuous">
     <parent link="base_link"/>
@@ -149,4 +160,5 @@
     <limit effort="100" velocity="10.0"/>
   </joint>
+  <!-- Right Wheel Joint (continuous rotation for locomotion) -->
   <joint name="right_wheel_joint" type="continuous">
     <parent link="base_link"/>
@@ -156,4 +168,5 @@
     <limit effort="100" velocity="10.0"/>
   </joint>
+  <!-- Caster Wheel Joint (fixed orientation, free to roll) -->
   <joint name="caster_joint" type="fixed">
     <parent link="base_link"/>
@@ -161,4 +174,5 @@
     <origin xyz="0.8 0 -0.2" rpy="0 0 0"/>
   </joint>
+  <!-- Camera Mounting Joint -->
   <joint name="camera_joint" type="fixed">
     <parent link="base_link"/>
@@ -166,4 +180,5 @@
     <origin xyz="0.9 0 0.36" rpy="0 0 0"/>
   </joint>
+  <!-- Camera Optical Frame Transformation (ROS standard camera frame alignment) -->
   <joint type="fixed" name="camera_optical_joint">
     <origin xyz="0 0 0" rpy="-${PI/2} 0 -${PI/2}"/>
